Commit message: Model modification in accordance with the issue/enchancement https://github.com/roboticslab-uc3m/teo-main/issues/28#.

File: teo_description/robots/teo.urdf (robot description, URDF)
Before this commit: robot teo, 30 links, 29 joints
Links:
- added link head_pitch_link, mass 1.0; collision mesh filename=package://teo_description/meshes/head/head.stl; visual mesh filename=package://teo_description/meshes/head/head.stl
- added link head_yaw_link, mass 1.0; collision mesh filename=package://teo_description/meshes/head/neck.stl; visual mesh filename=package://teo_description/meshes/head/neck.stl
- link waist_pitch_link: geometry collision mesh filename=package://teo_description/meshes/torso/L-torso-shoulder.stl; collision mesh filename=package://teo_description/meshes/torso/R-torso-shoulder.stl
Joints:
- removed joint base_joint
- added joint base_waist: type fixed, parent world, child waist, origin xyz=0 0 0 rpy=0 0 0
- added joint head_pitch: type revolute, parent head_yaw_link, child head_pitch_link, origin xyz=0 0 0.13 rpy=0 0 0, axis 0 1 0, limit lower=-1.27409035396 upper=1.27409035396 effort=30.0 velocity=3.0
- added joint head_yaw: type revolute, parent waist_pitch_link, child head_yaw_link, origin xyz=0 0 0.305 rpy=0 0 0, axis 0 0 1, limit lower=-0.506145483078 upper=0.146607657168 effort=30.0 velocity=3.0
- joint l_ankle_pitch: limit lower=-0.349065850399 upper=0.349065850399 effort=85.0 velocity=4.0 -> lower=-0.314159265359 upper=0.349065850399 effort=85.0 velocity=4.0; origin xyz=0 -0.033 -0.3 rpy=0 0 0 -> xyz=0 -0.0175 -0.3 rpy=0 0 0
- joint l_ankle_roll: axis 1 0 0 -> -1 0 0; limit lower=-1.4835298642 upper=1.4835298642 effort=65.0 velocity=4.0 -> lower=-0.436332312999 upper=0.436332312999 effort=65.0 velocity=4.0
- joint l_elbow_pitch: axis 0 1 0 -> 0 1.0 0; limit lower=-1.74532925199 upper=1.74532925199 effort=30.0 velocity=3.0 -> lower=-1.74532925199 upper=0.174532925199 effort=30.0 velocity=3.0
- joint l_hip_pitch: limit lower=-2.09439510239 upper=0.785398163397 effort=60.0 velocity=4.0 -> lower=-0.523598775598 upper=0.785398163397 effort=60.0 velocity=4.0
- joint l_hip_roll: axis 1 0 0 -> -1 0 0; limit lower=-0.698131700798 upper=0.523598775598 effort=65.0 velocity=4.0 -> lower=-0.349065850399 upper=0.349065850399 effort=65.0 velocity=4.0
- joint l_hip_yaw: axis 0 0 1 -> 0 0 1.0; limit lower=-0.523598775598 upper=0.418879020479 effort=45.0 velocity=4.0 -> lower=-1.57079632679 upper=1.57079632679 effort=45.0 velocity=4.0; origin xyz=0 0.146 -0.10237 rpy=0 0 0 -> xyz=0 0.146 -0.092 rpy=0 0 0
- joint l_knee_pitch: limit lower=0.0 upper=1.57079632679 effort=140.0 velocity=4.0 -> lower=-0.0872664625997 upper=1.3962634016 effort=140.0 velocity=4.0
- joint l_shoulder_pitch: axis 0 1 0 -> 0 1.0 0; limit lower=-3.14159265359 upper=3.14159265359 effort=30.0 velocity=3.0 -> lower=-1.2217304764 upper=0.785398163397 effort=30.0 velocity=3.0; origin xyz=-0.0 0.34 0.305 rpy=0 0 0 -> xyz=-0.0 0.34692 0 rpy=0 0 0; parent waist_pitch_link -> head_yaw_link
- joint l_shoulder_roll: limit lower=-0.785398163397 upper=2.09439510239 effort=30.0 velocity=3.0 -> lower=-0.261799387799 upper=1.2217304764 effort=30.0 velocity=3.0
- joint l_shoulder_yaw: axis 0 0 1 -> 0 0 -1; limit lower=-1.0471975512 upper=1.0471975512 effort=30.0 velocity=3.0 -> lower=-1.308996939 upper=0.174532925199 effort=30.0 velocity=3.0
- joint l_wrist_pitch: axis 0 1 0 -> 0 1.0 0; limit lower=-0.698131700798 upper=0.959931088597 effort=30.0 velocity=3.0 -> lower=-1.74532925199 upper=0.174532925199 effort=30.0 velocity=3.0
- joint l_wrist_yaw: axis 0 0 1 -> 0 0 -1; limit lower=-1.83259571459 upper=1.83259571459 effort=30.0 velocity=3.0 -> lower=-1.57079632679 upper=1.57079632679 effort=30.0 velocity=3.0
- joint r_ankle_pitch: limit lower=-0.349065850399 upper=0.349065850399 effort=85.0 velocity=4.0 -> lower=-0.314159265359 upper=0.349065850399 effort=85.0 velocity=4.0; origin xyz=0 0.033 -0.3 rpy=0 0 0 -> xyz=0 0.0175 -0.3 rpy=0 0 0
- joint r_ankle_roll: axis 1 0 0 -> -1 0 0; limit lower=-1.4835298642 upper=1.4835298642 effort=65.0 velocity=4.0 -> lower=-0.436332312999 upper=0.436332312999 effort=65.0 velocity=4.0
- joint r_elbow_pitch: axis 0 1 0 -> 0 -1.0 0; limit lower=-1.74532925199 upper=1.74532925199 effort=30.0 velocity=3.0 -> lower=-0.174532925199 upper=1.74532925199 effort=30.0 velocity=3.0
- joint r_hip_pitch: limit lower=-2.09439510239 upper=0.785398163397 effort=60.0 velocity=4.0 -> lower=-0.523598775598 upper=0.785398163397 effort=60.0 velocity=4.0
- joint r_hip_roll: axis 1 0 0 -> -1 0 0; limit lower=-0.698131700798 upper=0.523598775598 effort=65.0 velocity=4.0 -> lower=-0.349065850399 upper=0.349065850399 effort=65.0 velocity=4.0
- joint r_hip_yaw: axis 0 0 1 -> 0 0 -1.0; limit lower=-0.523598775598 upper=0.418879020479 effort=45.0 velocity=4.0 -> lower=-1.57079632679 upper=1.57079632679 effort=45.0 velocity=4.0; origin xyz=0 -0.146 -0.10237 rpy=0 0 0 -> xyz=0 -0.146 -0.092 rpy=0 0 0
- joint r_knee_pitch: limit lower=0.0 upper=1.57079632679 effort=140.0 velocity=4.0 -> lower=-0.0872664625997 upper=1.3962634016 effort=140.0 velocity=4.0
- joint r_shoulder_pitch: axis 0 1 0 -> 0 -1.0 0; limit lower=-3.14159265359 upper=3.14159265359 effort=30.0 velocity=3.0 -> lower=-0.785398163397 upper=1.2217304764 effort=30.0 velocity=3.0; origin xyz=-0.0 -0.34 0.305 rpy=0 0 0 -> xyz=-0.0 -0.34692 0 rpy=0 0 0; parent waist_pitch_link -> head_yaw_link
- joint r_shoulder_roll: limit lower=-0.785398163397 upper=2.09439510239 effort=30.0 velocity=3.0 -> lower=-1.2217304764 upper=0.261799387799 effort=30.0 velocity=3.0
- joint r_shoulder_yaw: axis 0 0 1 -> 0 0 -1; limit lower=-1.0471975512 upper=1.0471975512 effort=30.0 velocity=3.0 -> lower=-0.174532925199 upper=1.308996939 effort=30.0 velocity=3.0
- joint r_wrist_pitch: axis 0 1 0 -> 0 -1.0 0; limit lower=-0.698131700798 upper=0.959931088597 effort=30.0 velocity=3.0 -> lower=-0.174532925199 upper=1.74532925199 effort=30.0 velocity=3.0
- joint r_wrist_yaw: axis 0 0 1 -> 0 0 -1; limit lower=-1.83259571459 upper=1.83259571459 effort=30.0 velocity=3.0 -> lower=-1.57079632679 upper=1.57079632679 effort=30.0 velocity=3.0
- joint waist_pitch: limit lower=-0.785398163397 upper=0.523598775598 effort=30.0 velocity=3.0 -> lower=-0.174532925199 upper=0.174532925199 effort=30.0 velocity=3.0
- joint waist_yaw: limit lower=-0.785398163397 upper=0.523598775598 effort=30.0 velocity=3.0 -> lower=-0.785398163397 upper=0.785398163397 effort=30.0 velocity=3.0; origin xyz=0.0 0 0.1907 rpy=0 0 0 -> xyz=0.0 0 0.1932 rpy=0 0 0

File: teo_description/robots/teo_humanoid.urdf.xacro (robot description, xacro)
@@ -21,4 +21,5 @@
   <!--xacro:include filename="$(find teo_description)/urdf/visual.xacro" /-->
   <xacro:include filename="$(find teo_description)/urdf/others/teo_colors.xacro" />
+  <xacro:include filename="$(find teo_description)/urdf/head/head_vis.urdf.xacro" />
   <xacro:include filename="$(find teo_description)/urdf/torso/torso_vis.urdf.xacro" />
   <xacro:include filename="$(find teo_description)/urdf/legs/legs_vis.urdf.xacro" />

File: teo_description/robots/teo_humanoid_attach.urdf.xacro (robot description, xacro)
@@ -2,5 +2,5 @@
 <!--
   ROS urdf definition of TEO humanoid robot
-  Author: Domingo Esteban
+  Author: Domingo Esteban, Raul Fernandez Fernandez
   RoboticsLab, Universidad Carlos III de Madrid
   This file loads TEO model with a basic visualization.
@@ -21,4 +21,5 @@
   <!--xacro:include filename="$(find teo_description)/urdf/visual.xacro" /-->
   <xacro:include filename="$(find teo_description)/urdf/others/teo_colors.xacro" />
+  <xacro:include filename="$(find teo_description)/urdf/head/head_vis.urdf.xacro" />
   <xacro:include filename="$(find teo_description)/urdf/torso/torso_vis.urdf.xacro" />
   <xacro:include filename="$(find teo_description)/urdf/legs/legs_vis.urdf.xacro" />

File: teo_description/urdf/arms/arm.urdf.xacro (robot description, xacro)
@@ -10,23 +10,21 @@
 <!-- *** TEO ARM PARAMETERS -->
 <!-- Link lengths (meters)-->
-	<!--xacro:property name="chest_link1" value="0.0" />
-	<xacro:property name="chest_link2" value="0.245" /-->
-	<xacro:property name="arm_link1" value="0.340" /> <!-- Clavicle -->
+	<xacro:property name="arm_link1" value="0.34692" /> <!-- Clavicle -->
 	<xacro:property name="arm_link2" value="0.32901" /> <!-- Humerus -->
 	<xacro:property name="arm_link3" value="0.202" /> <!-- Ulna -->
-<!-- Minimum angles (degrees) -->
-	<xacro:property name="shoulder_pitch_lower" value="${-180 * deg_to_rad}" />
-	<xacro:property name="shoulder_roll_lower" value="${-45 * deg_to_rad}" />
-	<xacro:property name="shoulder_yaw_lower" value="${-60 * deg_to_rad}" />
-	<xacro:property name="elbow_pitch_lower" value="${-100 * deg_to_rad}" />
-	<xacro:property name="wrist_yaw_lower" value="${-105 * deg_to_rad}" />
-	<xacro:property name="wrist_pitch_lower" value="${-40 * deg_to_rad}" />
-<!-- Maximum angles (degrees) -->
-	<xacro:property name="shoulder_pitch_upper" value="${180 * deg_to_rad}" />
-	<xacro:property name="shoulder_roll_upper" value="${120 * deg_to_rad}" />
-	<xacro:property name="shoulder_yaw_upper" value="${60 * deg_to_rad}" />
+<!-- Minimum angles right arm  (degrees) -->
+	<xacro:property name="shoulder_pitch_lower" value="${-45 * deg_to_rad}" />
+	<xacro:property name="shoulder_roll_lower" value="${-70 * deg_to_rad}" />
+	<xacro:property name="shoulder_yaw_lower" value="${-10 * deg_to_rad}" />
+	<xacro:property name="elbow_pitch_lower" value="${-10 * deg_to_rad}" />
+	<xacro:property name="wrist_yaw_lower" value="${-90 * deg_to_rad}" />
+	<xacro:property name="wrist_pitch_lower" value="${-10 * deg_to_rad}" />
+<!-- Maximum angles right arm (degrees) -->
+	<xacro:property name="shoulder_pitch_upper" value="${70 * deg_to_rad}" />
+	<xacro:property name="shoulder_roll_upper" value="${15 * deg_to_rad}" />
+	<xacro:property name="shoulder_yaw_upper" value="${75 * deg_to_rad}" />
 	<xacro:property name="elbow_pitch_upper" value="${100 * deg_to_rad}" />
-	<xacro:property name="wrist_yaw_upper" value="${105 * deg_to_rad}" />
-	<xacro:property name="wrist_pitch_upper" value="${55 * deg_to_rad}" />
+	<xacro:property name="wrist_yaw_upper" value="${90 * deg_to_rad}" />
+	<xacro:property name="wrist_pitch_upper" value="${100 * deg_to_rad}" />
 <!-- Effort limit of the angles -->
 	<xacro:property name="shoulder_pitch_effort" value="30.0" />
@@ -69,11 +67,7 @@
     <link name="${side}_shoulder_pitch_link">
       <inertial>
-        <!-- <origin xyz="-0.002758 ${reflect*0.020318} 0.011855" rpy="0 0 0"/> -->
 	<origin xyz="0.0 ${reflect*0.0} 0.0" rpy="0 0 0"/>
         <mass value="0.005"/>
-        <!-- <inertia ixx="1.000" ixy="0.000" ixz="0.000" iyy="1.000" iyz="0.000" izz="1.000" />-->
 	<inertia ixx="0.059121e-2" ixy="0.000603e-2" ixz="0.000103e-2" iyy="0.024956e-2" iyz="0.005131e-2" izz="0.050653e-2" />
-	<!-- Mass scaled-->
-	<!-- <inertia ixx="0.295605e-5" ixy="0.003015e-5" ixz="0.000515e-5" iyy="0.12478e-5" iyz="0.025655e-5" izz="0.253265e-5" /> -->
       </inertial>
       <xacro:insert_visualization_shoulder_pitch side="${side}" reflect="${reflect}"/>
@@ -81,14 +75,7 @@
     <link name="${side}_shoulder_roll_link">
       <inertial>
-        <!-- <origin xyz="-0.006929 ${reflect*-0.010231} -0.034506" rpy="0 0 0"/> -->
 	<origin xyz="0.0 ${reflect*0.0} 0.0" rpy="0 0 0"/>
         <mass value="0.005"/>
-        <!-- <inertia
-				  ixx="1.000" ixy="0.000" ixz="0.000"
-					iyy="1.000" iyz="0.000"
-					izz="1.000" /> -->
 	<inertia ixx="0.018036e-2" ixy="-0.000773e-2" ixz="0.002406e-2" iyy="0.024499e-2" iyz="0.001826e-2" izz="0.013143e-2" />
-	<!-- Mass escaled -->
-	<!-- <inertia ixx="0.09018e-5" ixy="-0.003865e-5" ixz="0.01203e-5" iyy="0.122495e-5" iyz="0.00913e-5" izz="0.065715e-5" /> -->
       </inertial>
       <xacro:insert_visualization_shoulder_roll side="${side}" reflect="${reflect}"/>
@@ -96,14 +83,7 @@
     <link name="${side}_shoulder_yaw_link">
       <inertial>
-        <!-- <origin xyz="0.003730 ${reflect*0.000060} 0.062982" rpy="0 0 0"/> -->
 	<origin xyz="0.0 ${reflect*0.0} 0.0" rpy="0 0 0"/>
         <mass value="1.750625"/>
-        <!-- <inertia
-				  ixx="7.000e-3" ixy="2.148e-5" ixz="3.931e-5"
-					iyy="7.000e-3" iyz="1.558e-5"
-					izz="8.195e-4" /> -->
 	<inertia ixx="0.227681e-2" ixy="0.0" ixz="0.0" iyy="0.224821e-2" iyz="-0.000684e-2" izz="0.032283e-2" />
-	<!-- Mass scaled -->
-	<!-- <inertia ixx="0.39844175e-2" ixy="0.0" ixz="0.0" iyy="0.39343675e-2" iyz="-0.001197e-2" izz="0.05649525e-2" /> -->
       </inertial>
       <xacro:insert_visualization_shoulder_yaw side="${side}" reflect="${reflect}"/>
@@ -113,11 +93,5 @@
         <origin xyz="0.0 ${reflect*0.001} -0.000588" rpy="0 0 0"/>
         <mass value="2.396"/>
-        <!-- <inertia
-				  ixx="3.000e-3" ixy="9.570e-4" ixz="6.522e-6"
-					iyy="3.000e-3" iyz="3.778e-5"
-					izz="3.000e-3" /> -->
 	<inertia ixx="0.059390e-2" ixy="0.0" ixz="0.0" iyy="0.060871e-2" iyz="-0.0" izz="0.023257e-2" /> -->
-	<!-- Mass scaled-->
-	<!-- <inertia ixx="0.14229844e-2" ixy="0.0" ixz="0.0" iyy="0.145846916e-2" iyz="-0.0" izz="0.055723772e-2" />-->
       </inertial>
       <xacro:insert_visualization_elbow_pitch side="${side}" reflect="${reflect}"/>
@@ -127,12 +101,5 @@
         <origin xyz="-0.004657 ${reflect*-0.001356} 0.035884" rpy="0 0 0"/>
         <mass value="0.005"/>
-        <!-- <inertia
-				  ixx="1.000" ixy="0.000" ixz="0.000"
-					iyy="1.000" iyz="0.000"
-					izz="1.000" /> -->
-	<!--<inertia ixx="5*0.004543e-8" ixy="5*0.000068e-8" ixz="5*0.000070e-8" iyy="5*0.003969e-8" iyz="5*-0.000074e-8" izz="5*0.002118e-8" /> -->
 	<inertia ixx="0.004543e-2" ixy="0.000068e-2" ixz="0.000070e-2" iyy="0.003969e-2" iyz="-0.000074e-2" izz="0.002118e-2" />
-	<!-- Mass scaled -->
-	<!-- <inertia ixx="0.022715e-5" ixy="0.00034e-5" ixz="0.00035e-5" iyy="0.019845e-5" iyz="-0.00037e-5" izz="0.01059e-5" /> -->
       </inertial>
       <xacro:insert_visualization_wrist_yaw side="${side}" reflect="${reflect}"/>
@@ -142,13 +109,5 @@
         <origin xyz="-0.002438 ${reflect*0.004651} -0.044838" rpy="0 0 0"/>
         <mass value="0.3"/>
-        <!-- <inertia
-				  ixx="3.400e-4" ixy="0.000" ixz="0.000"
-					iyy="3.125e-4" iyz="0.000"
-					izz="1.525e-4" />-->
-	<!--<inertia ixx="0.007270e-2" ixy="0.0" ixz="0.0" iyy="0.007586e-2" iyz="0.000055e-2" izz="0.003248e-2" /> -->
-	<!--<inertia ixx="-0.008337e-2" ixy="0.003468e-2" ixz="-0.005567e-2" iyy="-0.013674e-2" iyz="0.005108e-2" izz="0.005142e-2" /> -->
 	<inertia ixx="1.0e-2" ixy="0.0" ixz="0.0" iyy="1.0e-2" iyz="0.0" izz="1.0e-2" />
-	<!-- Mass scaled -->
-	<!-- <inertia ixx="-0.02502e-2" ixy="0.010401e-2" ixz="-0.016707e-2" iyy="-0.041034e-2" iyz="0.01146e-2" izz="0.015405e-2" /> -->
       </inertial>
       <xacro:insert_visualization_wrist_pitch side="${side}" reflect="${reflect}"/>
@@ -156,11 +115,16 @@
   </xacro:macro>
   <!-- Joints -->
-  <xacro:macro name="arms_joints" params="side reflect effortTransmission velocityTransmission positionTransmission">
+  <xacro:macro name="arms_joints" params="side reflect effortTransmission velocityTransmission positionTransmission right">
     <joint name="${side}_shoulder_pitch" type="revolute">
-      <parent link="waist_pitch_link"/>
+      <parent link="head_yaw_link"/>
       <child link="${side}_shoulder_pitch_link"/>
-      <origin xyz="-${chest_link1} ${reflect*arm_link1} ${chest_link2+torso_link2}" rpy="0 0 0"/>
-      <axis xyz="0 1 0"/>
+      <origin xyz="-${chest_link1} ${reflect*arm_link1} 0" rpy="0 0 0"/>
+      <axis xyz="0 ${reflect*1} 0"/>
+      <xacro:if value="${right}">
       <limit velocity="${shoulder_pitch_velocity}" effort="${shoulder_pitch_effort}" lower="${shoulder_pitch_lower}" upper="${shoulder_pitch_upper}"/>
+      </xacro:if>
+      <xacro:unless value="${right}">
+      <limit velocity="${shoulder_pitch_velocity}" effort="${shoulder_pitch_effort}" lower="${-shoulder_pitch_upper}" upper="${-shoulder_pitch_lower}"/>
+      </xacro:unless>
     </joint>
     <joint name="${side}_shoulder_roll" type="revolute">
@@ -169,5 +133,10 @@
       <origin xyz="0 0 0" rpy="0 0 0"/>
       <axis xyz="1 0 0"/>
+      <xacro:if value="${right}">
       <limit velocity="${shoulder_roll_velocity}" effort="${shoulder_roll_effort}" lower="${shoulder_roll_lower}" upper="${shoulder_roll_upper}"/>
+      </xacro:if>
+      <xacro:unless value="${right}">
+      <limit velocity="${shoulder_roll_velocity}" effort="${shoulder_roll_effort}" lower="${-shoulder_roll_upper}" upper="${-shoulder_roll_lower}"/>
+      </xacro:unless>
     </joint>
     <joint name="${side}_shoulder_yaw" type="revolute">
@@ -175,6 +144,11 @@
       <child link="${side}_shoulder_yaw_link"/>
       <origin xyz="0 0 0" rpy="0 0 0"/>
-      <axis xyz="0 0 1"/>
+      <axis xyz="0 0 -1"/>
+      <xacro:if value="${right}">
       <limit velocity="${shoulder_yaw_velocity}" effort="${shoulder_yaw_effort}" lower="${shoulder_yaw_lower}" upper="${shoulder_yaw_upper}"/>
+      </xacro:if>
+      <xacro:unless value="${right}">
+      <limit velocity="${shoulder_yaw_velocity}" effort="${shoulder_yaw_effort}" lower="${-shoulder_yaw_upper}" upper="${-shoulder_yaw_lower}"/>
+      </xacro:unless>
     </joint>
     <joint name="${side}_elbow_pitch" type="revolute">
@@ -182,6 +156,11 @@
       <child link="${side}_elbow_pitch_link"/>
       <origin xyz="0 0 -${arm_link2}" rpy="0 0 0"/>
-      <axis xyz="0 1 0"/>
+      <axis xyz="0 ${reflect*1} 0"/>
+      <xacro:if value="${right}">
       <limit velocity="${elbow_pitch_velocity}" effort="${elbow_pitch_effort}" lower="${elbow_pitch_lower}" upper="${elbow_pitch_upper}"/>
+      </xacro:if>
+      <xacro:unless value="${right}">
+      <limit velocity="${elbow_pitch_velocity}" effort="${elbow_pitch_effort}" lower="${-elbow_pitch_upper}" upper="${-elbow_pitch_lower}"/>
+      </xacro:unless>
     </joint>
     <joint name="${side}_wrist_yaw" type="revolute">
@@ -189,6 +168,11 @@
       <child link="${side}_wrist_yaw_link"/>
       <origin xyz="0 0 -${arm_link3}" rpy="0 0 0"/>
-      <axis xyz="0 0 1"/>
+      <axis xyz="0 0 -1"/>
+      <xacro:if value="${right}">
       <limit velocity="${wrist_yaw_velocity}" effort="${wrist_yaw_effort}" lower="${wrist_yaw_lower}" upper="${wrist_yaw_upper}"/>
+      </xacro:if>
+      <xacro:unless value="${right}">
+      <limit velocity="${wrist_yaw_velocity}" effort="${wrist_yaw_effort}" lower="${-wrist_yaw_upper}" upper="${-wrist_yaw_lower}"/>
+      </xacro:unless>
     </joint>
     <joint name="${side}_wrist_pitch" type="revolute">
@@ -196,6 +180,11 @@
       <child link="${side}_wrist_pitch_link"/>
       <origin xyz="0 0 0" rpy="0 0 0"/>
-      <axis xyz="0 1 0"/>
+      <axis xyz="0 ${reflect*1} 0"/>
+      <xacro:if value="${right}">
       <limit velocity="${wrist_pitch_velocity}" effort="${wrist_pitch_effort}" lower="${wrist_pitch_lower}" upper="${wrist_pitch_upper}"/>
+      </xacro:if>
+      <xacro:unless value="${right}">
+      <limit velocity="${wrist_pitch_velocity}" effort="${wrist_pitch_effort}" lower="${-wrist_pitch_upper}" upper="${-wrist_pitch_lower}"/>
+      </xacro:unless>
     </joint>
     <xacro:limb_joint_simple_transmission name="shoulder" side="${side}" axis="pitch" reduction="${shoulder_pitch_reduction}" effortTransmission="${effortTransmission}" velocityTransmission="${velocityTransmission}" positionTransmission="${positionTransmission}"/>
@@ -206,7 +195,7 @@
     <xacro:limb_joint_simple_transmission name="wrist" side="${side}" axis="pitch" reduction="${wrist_pitch_reduction}" effortTransmission="${effortTransmission}" velocityTransmission="${velocityTransmission}" positionTransmission="${positionTransmission}"/>
   </xacro:macro>
-  <xacro:arms_links side="l" reflect="1"/>
+  <xacro:arms_links side="l" reflect="1" />
   <xacro:arms_links side="r" reflect="-1"/>
-  <xacro:arms_joints side="l" reflect="1" effortTransmission="0" velocityTransmission="0" positionTransmission="1"/>
-  <xacro:arms_joints side="r" reflect="-1" effortTransmission="0" velocityTransmission="0" positionTransmission="1"/>
+  <xacro:arms_joints side="l" reflect="1" effortTransmission="0" velocityTransmission="0" positionTransmission="1" right="0"/>
+  <xacro:arms_joints side="r" reflect="-1" effortTransmission="0" velocityTransmission="0" positionTransmission="1" right="1"/>
 </robot>
