Commit message: Model modification in accordance with the issue/enchancement https://github.com/roboticslab-uc3m/teo-main/issues/28#.

File: teo_description/urdf/legs/leg.urdf.xacro (robot description, xacro)
@@ -13,24 +13,24 @@
   <xacro:property name="prop_kg_tibia_vol_unit" value="2638.403042" /> <!-- Relation Kg - Volume Unit -->
 <!-- Link lengths -->
-	<xacro:property name="leg_link0" value="0.10237" /> <!-- Hip -->
+	<xacro:property name="leg_link0" value="0.092" /> <!-- Hip -->
 	<xacro:property name="leg_link1" value="0.146" /> <!-- Hip -->
 	<xacro:property name="leg_link2" value="0.33" /> <!-- Femur -->
 	<xacro:property name="leg_link3" value="0.3" /> <!-- Tibia -->
-	<xacro:property name="leg_link4" value="0.033" /> <!-- Patella -->
+	<xacro:property name="leg_link4" value="0.0175" /> <!-- Patella -->
 	<xacro:property name="leg_link5" value="0.124" /> <!-- Astragalus -->
-<!-- Minimum angles -->
-	<xacro:property name="hip_yaw_lower" value="${-30 * deg_to_rad}" />
-	<xacro:property name="hip_roll_lower" value="${-40 * deg_to_rad}" />
-	<xacro:property name="hip_pitch_lower" value="${-120 * deg_to_rad}" />
-	<xacro:property name="knee_pitch_lower" value="${0 * deg_to_rad}" />
-	<xacro:property name="ankle_pitch_lower" value="${-20 * deg_to_rad}" />
-	<xacro:property name="ankle_roll_lower" value="${-85 * deg_to_rad}" />
-<!-- Maximum angles -->
-	<xacro:property name="hip_yaw_upper" value="${24 * deg_to_rad}" />
-	<xacro:property name="hip_roll_upper" value="${30 * deg_to_rad}" />
+<!-- Minimum angles right leg -->
+	<xacro:property name="hip_yaw_lower" value="${-90 * deg_to_rad}" />
+	<xacro:property name="hip_roll_lower" value="${-20 * deg_to_rad}" />
+	<xacro:property name="hip_pitch_lower" value="${-30 * deg_to_rad}" />
+	<xacro:property name="knee_pitch_lower" value="${-5 * deg_to_rad}" />
+	<xacro:property name="ankle_pitch_lower" value="${-18 * deg_to_rad}" />
+	<xacro:property name="ankle_roll_lower" value="${-25 * deg_to_rad}" />
+<!-- Maximum angles right leg -->
+	<xacro:property name="hip_yaw_upper" value="${90 * deg_to_rad}" />
+	<xacro:property name="hip_roll_upper" value="${20 * deg_to_rad}" />
 	<xacro:property name="hip_pitch_upper" value="${45 * deg_to_rad}" />
-	<xacro:property name="knee_pitch_upper" value="${90 * deg_to_rad}" />
+	<xacro:property name="knee_pitch_upper" value="${80 * deg_to_rad}" />
 	<xacro:property name="ankle_pitch_upper" value="${20 * deg_to_rad}" />
-	<xacro:property name="ankle_roll_upper" value="${85 * deg_to_rad}" />
+	<xacro:property name="ankle_roll_upper" value="${25 * deg_to_rad}" />
 <!-- Effort limit of the angles -->
 	<xacro:property name="hip_yaw_effort" value="45.0" />
@@ -74,8 +74,5 @@
       <inertial>
         <origin xyz="0.0 ${-reflect*0.0} 0.0" rpy="0 0 0"/>
-        <!-- <mass value="0.001"/> -->
-        <mass value="1.0"/>
-        <!-- <mass value="${prop_kg_motor_vol_unit*0.000185}"/> -->
-        <!-- <inertia ixx="3.4076E-4" ixy="${-reflect*0.0}" ixz="5.4E-7" iyy="5.7638E-4" iyz="${-reflect*3.7186E-4}" izz="0.84231334"/> -->
+        <mass value="1.0"/>
 	<inertia ixx="3.4076E-4" ixy="${-reflect*0.0}" ixz="5.4E-7" iyy="5.7638E-4" iyz="${-reflect*0.0}" izz="0.037186e-2"/>
       </inertial>
@@ -85,8 +82,5 @@
       <inertial>
         <origin xyz="0.0 ${-reflect*0.0} -0.017753" rpy="0 0 0"/>
-        <!-- <origin xyz="-0.029398 ${-reflect*0.001062} -0.017753" rpy="0 0 0"/> -->
-        <!-- <mass value="0.001"/> -->
-        <mass value="1.0"/>
-        <!-- <mass value="${prop_kg_motor_vol_unit*0.000317}"/> -->
+        <mass value="1.0"/>
         <inertia ixx="3.6847E-4" ixy="${-reflect*4.34E-6}" ixz="1.0E-8" iyy="1.9052E-4" iyz="${-reflect*0.0}" izz="4.5536E-4"/>
       </inertial>
@@ -96,10 +90,6 @@
       <inertial>
         <origin xyz="0.0 ${-reflect*0.0} ${-0.172570}" rpy="0 0 0"/>
-        <!-- <origin xyz="${-0.013877} ${-reflect*0.0} ${-0.172570}" rpy="0 0 0"/> -->
-        <!-- <mass value="1.844"/> -->
-        <mass value="1.0"/>
-        <!-- <mass value="${prop_kg_femur_vol_unit*0.005587}"/> -->
+        <mass value="1.0"/>
         <inertia ixx="4.453648E-2" ixy="${-reflect*-1.0E-8}" ixz="0.00130498" iyy="4.46349E-2" iyz="${-reflect*4.0E-8}" izz="2.207083E-2"/>
-        <!-- <inertia ixx="4.453648E-5" ixy="${-reflect*-1.0E-11}" ixz="0.00000130498" iyy="4.46349E-5" iyz="${-reflect*3.0E-11}" izz="2.207083E-5"/> -->
       </inertial>
       <xacro:insert_visualization_femur_link side="${side}" reflect="${reflect}"/>
@@ -107,10 +97,6 @@
     <link name="${side}_tibia_link">
       <inertial>
-        <!-- <origin xyz="${-0.013-0.001019} ${-reflect*(-(leg_link4)+0.024670)} ${-leg_link3+0.127850}" rpy="0 0 0"/> -->
         <origin xyz="0.0 ${-reflect*0.0} -0.142721" rpy="0 0 0"/>
-        <!-- <origin xyz="${-0.010351} ${-reflect*0.0} -0.142721" rpy="0 0 0"/> -->
-        <!-- <mass value="2.0817"/> -->
-        <mass value="1.0"/>
-        <!-- <mass value="${prop_kg_femur_vol_unit*0.005587}"/> -->
+        <mass value="1.0"/>
         <inertia ixx="4.644211E-2" ixy="${-reflect*0.0}" ixz="-7.32E-6" iyy="4.548272E-2" iyz="${-reflect*-1.0E-8}" izz="8.16616E-3"/>
       </inertial>
@@ -120,11 +106,6 @@
       <inertial>
         <origin xyz="0.0 ${-reflect*0.0} 0.028198" rpy="0 0 0"/>
-        <!-- <origin xyz="0.004952 ${-reflect*-0.005263} 0.028198" rpy="0 0 0"/> -->
-        <mass value="1.0"/>
-        <!-- <mass value="1.0"/> -->
-        <!-- <inertia ixx="0.00082035023" ixy="${-reflect*0.00000048534}" ixz="0.00000226301" iyy="0.00082074105" iyz="${-reflect*-0.00002892247}" izz="0.00037614067"/> -->
+        <mass value="1.0"/>
 	<inertia ixx="0.010237e-2" ixy="${-reflect*0.000014}" ixz="0.0" iyy="0.035107e-2" iyz="${-reflect*-0.0}" izz="0.035006e-2"/>
-        <!-- REVISAR ESTE!! que falla -->
-        <!-- <inertia ixx="3.3782E-7" ixy="${-reflect*-1.65E-9}" ixz="0.0" iyy="3.8475E-7" iyz="${-reflect*0.0}" izz="5.8551E-7"/> -->
       </inertial>
       <xacro:insert_visualization_ankle_pitch side="${side}" reflect="${reflect}"/>
@@ -133,10 +114,6 @@
       <inertial>
         <origin xyz="0.0 ${-reflect*0.0} -0.042127" rpy="0 0 0"/>
-        <!-- <origin xyz="-0.006788 ${-reflect*0.000020} -0.042127" rpy="0 0 0"/> -->
-        <mass value="1.0"/>
-        <!-- <mass value="1.015338978"/> -->
+        <mass value="1.0"/>
         <inertia ixx="2.6324E-4" ixy="${-reflect*0.0}" ixz="7.4E-6" iyy="0.000571" iyz="${-reflect*0}" izz="4.633E-4"/>
-        <!-- REVISAR! -->
-        <!-- <inertia ixx="2.6324E-7" ixy="${-reflect*0.0}" ixz="7.4E-9" iyy="0.000000571" iyz="${-reflect*0}" izz="4.633E-7"/> -->
       </inertial>
       <xacro:insert_visualization_ankle_roll side="${side}" reflect="${reflect}"/>
@@ -145,8 +122,5 @@
       <inertial>
         <origin xyz="0.022629 ${-reflect*0.002448} 0.011325" rpy="0 0 0"/>
-        <!-- <origin xyz="0.022629 ${-reflect*0.002448} 0.011325" rpy="0 0 0"/> -->
-        <mass value="1.0"/>
-        <!-- <mass value="2.884061022"/> -->
-        <!--<inertia ixx="6.699E-4" ixy="${-reflect*-0.000093}" ixz="9.066E-5" iyy="1.69929E-3" iyz="${-reflect*7.08E-6}" izz="2.28359E-3"/> -->
+        <mass value="1.0"/>
 	<inertia ixx="0.065992e-2" ixy="${-reflect*0.010716e-2}" ixz="0.008960e-2" iyy="0.167825e-2" iyz="${-reflect*-0.000847e-2}" izz="0.225319e-2"/>
       </inertial>
@@ -160,8 +134,8 @@
       <parent link="waist"/>
       <child link="${side}_hip_yaw_link"/>
-      <origin xyz="0 ${reflect*leg_link1} ${-leg_link0}" rpy="0 0 0"/> <!--y=Leg_link1-->
-      <axis xyz="0 0 1"/>
+      <origin xyz="0 ${reflect*leg_link1} ${-leg_link0}" rpy="0 0 0"/>
+      <axis xyz="0 0 ${reflect*1}"/>
       <limit velocity="${hip_yaw_velocity}" effort="${hip_yaw_effort}" lower="${hip_yaw_lower}" upper="${hip_yaw_upper}"/>
-			<dynamics damping="${hip_yaw_damping}" friction="${hip_yaw_friction}"/>
+      <dynamics damping="${hip_yaw_damping}" friction="${hip_yaw_friction}"/>
     </joint>
     <joint name="${side}_hip_roll" type="revolute">
@@ -169,7 +143,7 @@
       <child link="${side}_hip_roll_link"/>
       <origin xyz="0 0 0" rpy="0 0 0"/>
-      <axis xyz="1 0 0"/>
+      <axis xyz="-1 0 0"/>
       <limit velocity="${hip_roll_velocity}" effort="${hip_roll_effort}" lower="${hip_roll_lower}" upper="${hip_roll_upper}"/>
-			<dynamics damping="${hip_roll_damping}" friction="${hip_roll_friction}"/>
+      <dynamics damping="${hip_roll_damping}" friction="${hip_roll_friction}"/>
     </joint>
     <joint name="${side}_hip_pitch" type="revolute">
@@ -179,5 +153,5 @@
       <axis xyz="0 1 0"/>
       <limit velocity="${hip_pitch_velocity}" effort="${hip_pitch_effort}" lower="${hip_pitch_lower}" upper="${hip_pitch_upper}"/>
-			<dynamics damping="${hip_pitch_damping}" friction="${hip_pitch_friction}"/>
+      <dynamics damping="${hip_pitch_damping}" friction="${hip_pitch_friction}"/>
     </joint>
     <joint name="${side}_knee_pitch" type="revolute">
@@ -187,5 +161,5 @@
       <axis xyz="0 1 0"/>
       <limit velocity="${knee_pitch_velocity}" effort="${knee_pitch_effort}" lower="${knee_pitch_lower}" upper="${knee_pitch_upper}"/>
-			<dynamics damping="${knee_pitch_damping}" friction="${knee_pitch_friction}"/>
+      <dynamics damping="${knee_pitch_damping}" friction="${knee_pitch_friction}"/>
     </joint>
     <joint name="${side}_ankle_pitch" type="revolute">
@@ -195,5 +169,5 @@
       <axis xyz="0 1 0"/>
       <limit velocity="${ankle_pitch_velocity}" effort="${ankle_pitch_effort}" lower="${ankle_pitch_lower}" upper="${ankle_pitch_upper}"/>
-			<dynamics damping="${ankle_pitch_damping}" friction="${ankle_pitch_friction}"/>
+      <dynamics damping="${ankle_pitch_damping}" friction="${ankle_pitch_friction}"/>
     </joint>
     <joint name="${side}_ankle_roll" type="revolute">
@@ -201,5 +175,5 @@
       <child link="${side}_astragalus_link"/>
       <origin xyz="0 0 0" rpy="0 0 0"/>
-      <axis xyz="1 0 0"/>
+      <axis xyz="-1 0 0"/>
       <limit velocity="${ankle_roll_velocity}" effort="${ankle_roll_effort}" lower="${ankle_roll_lower}" upper="${ankle_roll_upper}"/>
 			<dynamics damping="${ankle_roll_damping}" friction="${ankle_roll_friction}"/>

File: teo_description/urdf/teo_structure.gazebo.xacro (robot description, xacro)
@@ -26,4 +26,19 @@
 			<material>Gazebo/White</material>
 		</gazebo> -->
+	</xacro:macro>
+	<!-- ############### -->
+	<!-- # HEAD LINKS # -->
+	<!-- ############### -->
+  <xacro:macro name="gazebo_head" params="">
+		<gazebo reference="head_yaw_link">
+			<mu1>0.9</mu1>
+			<mu2>0.9</mu2>
+			<!-- <material>Gazebo/White</material> -->
+		</gazebo>
+		<gazebo reference="head_pitch_link">
+			<mu1>0.9</mu1>
+			<mu2>0.9</mu2>
+			<!-- <material>Gazebo/White</material> -->
+		</gazebo>
 	</xacro:macro>
 	<!-- ############## -->

File: teo_description/urdf/teo_structure.urdf.xacro (robot description, xacro)
@@ -30,4 +30,5 @@
  <!-- Definitions of parts of the robot body -->
  <xacro:include filename="$(find teo_description)/urdf/torso/torso.urdf.xacro" />
+ <xacro:include filename="$(find teo_description)/urdf/head/head.urdf.xacro" />
  <xacro:include filename="$(find teo_description)/urdf/legs/leg.urdf.xacro" />
  <xacro:include filename="$(find teo_description)/urdf/arms/arm.urdf.xacro" />
@@ -38,4 +39,5 @@
   <xacro:include filename="$(find teo_description)/urdf/teo_structure.gazebo.xacro" />
   <xacro:gazebo_torso/>
+  <xacro:gazebo_head/>
   <xacro:gazebo_legs_links side="l" reflect="1"/>
   <xacro:gazebo_legs_links side="r" reflect="-1"/>

File: teo_description/urdf/teo_structure_attach.urdf.xacro (robot description, xacro)
@@ -30,4 +30,5 @@
  <!-- Definitions of parts of the robot body -->
  <xacro:include filename="$(find teo_description)/urdf/torso/torso.urdf.xacro" />
+ <xacro:include filename="$(find teo_description)/urdf/head/head.urdf.xacro" />
  <xacro:include filename="$(find teo_description)/urdf/legs/leg.urdf.xacro" />
  <xacro:include filename="$(find teo_description)/urdf/arms/arm.urdf.xacro" />
@@ -38,4 +39,5 @@
   <xacro:include filename="$(find teo_description)/urdf/teo_structure.gazebo.xacro" />
   <xacro:gazebo_torso/>
+  <xacro:gazebo_head/>
   <xacro:gazebo_legs_links side="l" reflect="1"/>
   <xacro:gazebo_legs_links side="r" reflect="-1"/>

File: teo_description/urdf/torso/torso.urdf.xacro (robot description, xacro)
@@ -13,16 +13,16 @@
 	<xacro:property name="waist_link1" value="0.0" />
 	<!--xacro:property name="waist_link2" value="0.287" /-->
-	<xacro:property name="waist_link2" value="0.19070" />
+	<xacro:property name="waist_link2" value="0.1932" />
 	<xacro:property name="torso_link1" value="0.0" />
-	<!--xacro:property name="torso_link2" value="0.06" /-->
 	<xacro:property name="torso_link2" value="0.06" />
-  <xacro:property name="chest_link1" value="0.0" />
-  <xacro:property name="chest_link2" value="0.245" />
+  	<xacro:property name="chest_link1" value="0.0" />
+  	<xacro:property name="chest_link2" value="0.245" />
+	<xacro:property name="chest_link" value="0.305" />
 <!-- Minimum angles -->
 	<xacro:property name="waist_yaw_lower" value="${-45 * deg_to_rad}" />
-  <xacro:property name="waist_pitch_lower" value="${-45 * deg_to_rad}" />
+  <xacro:property name="waist_pitch_lower" value="${-10 * deg_to_rad}" />
 <!-- Maximum angles -->
-	<xacro:property name="waist_yaw_upper" value="${30 * deg_to_rad}" />
-	<xacro:property name="waist_pitch_upper" value="${30 * deg_to_rad}" />
+	<xacro:property name="waist_yaw_upper" value="${45 * deg_to_rad}" />
+	<xacro:property name="waist_pitch_upper" value="${10 * deg_to_rad}" />
 <!-- Effort limit of the angles -->
 	<xacro:property name="waist_yaw_effort" value="30.0" />
@@ -93,6 +93,6 @@
   <link name="waist_pitch_link" >
     <inertial>
-      <origin xyz="0.0 0.0 0.221233" rpy="0 0 0"/>
-      <!-- <origin xyz="0.038788 -0.000008 0.221233" rpy="0 0 0"/> -->
+      <origin xyz="0.038788 -0.000008 0.221233" rpy="0 0 0"/>
+      <!-- <origin xyz="0.0 -0.0 0.221233" rpy="0 0 0"/> -->
       <mass value="1.0"/>
       <!-- <inertia

File: teo_description/urdf/torso/torso_vis.urdf.xacro (robot description, xacro)
@@ -77,31 +77,5 @@
       </geometry>
     </collision>
-    <visual>
-      <origin xyz="0 0 0.346" rpy="0 0 0"/>
-      <geometry>
-        <mesh filename="package://teo_description/meshes/torso/neck.stl"/>
-      </geometry>
-      <material name="LightGrey"/>
-    </visual>
-    <collision>
-      <origin xyz="0 0 0.346" rpy="0 0 0"/>
-      <geometry>
-        <mesh filename="package://teo_description/meshes/torso/neck.stl"/>
-      </geometry>
-    </collision>
-    <visual>
-      <origin xyz="0 0 0.434" rpy="0 0 0"/>
-      <geometry>
-        <mesh filename="package://teo_description/meshes/torso/head.stl"/>
-      </geometry>
-      <material name="LightGrey"/>
-    </visual>
-    <collision>
-      <origin xyz="0 0 0.434" rpy="0 0 0"/>
-      <geometry>
-        <mesh filename="package://teo_description/meshes/torso/head.stl"/>
-      </geometry>
-    </collision>
-  </xacro:macro>
+    </xacro:macro>
   <xacro:macro name="insert_visualization_waist" params="">
     <visual>
