Commit message: Fixed head_vis problem

File: teo_description/urdf/head/head_vis.urdf.xacro (robot description, xacro)
@@ -12,5 +12,5 @@
         <mesh filename="package://teo_description/meshes/head/neck.stl"/>
       </geometry>
-      <material name="LightGrey"/>
+      <material name="teoGray"/>
     </visual>
     <collision>
@@ -27,5 +27,5 @@
         <mesh filename="package://teo_description/meshes/head/head.stl"/>
       </geometry>
-      <material name="LightGrey"/>
+      <material name="teoGray"/>
     </visual>
     <collision>
